File: Electronic Design/LED_board.sch (EAGLE design)
At the start: 12 parts

Commit message: Adding resistor values
Parts:
- R1, R2, R3, R4, R5: value (none) -> 270E
Changed lines of the file:
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@@
 <parts>
 <part name="JP1" library="pinhead" deviceset="PINHD-1X8" device=""/>
-<part name="R1" library="resistor" deviceset="R-EU_" device="R0805"/>
+<part name="R1" library="resistor" deviceset="R-EU_" device="R0805" value="270E"/>
 <part name="LED1" library="led" deviceset="LED" device="5MM"/>
 <part name="P+1" library="supply1" deviceset="+5V" device=""/>
 <part name="SUPPLY1" library="supply2" deviceset="GND" device=""/>
-<part name="R2" library="resistor" deviceset="R-EU_" device="R0805"/>
-<part name="R3" library="resistor" deviceset="R-EU_" device="R0805"/>
-<part name="R4" library="resistor" deviceset="R-EU_" device="R0805"/>
-<part name="R5" library="resistor" deviceset="R-EU_" device="R0805"/>
+<part name="R2" library="resistor" deviceset="R-EU_" device="R0805" value="270E"/>
+<part name="R3" library="resistor" deviceset="R-EU_" device="R0805" value="270E"/>
+<part name="R4" library="resistor" deviceset="R-EU_" device="R0805" value="270E"/>
+<part name="R5" library="resistor" deviceset="R-EU_" device="R0805" value="270E"/>
 <part name="LED2" library="led" deviceset="LED" device="5MM"/>
 <part name="LED3" library="led" deviceset="LED" device="5MM"/>

Commit message: changing resistors to 1206 size
Parts:
- R1, R2, R3, R4, R5: device resistor:R-EU_R0805 -> resistor:R-EU_R1206
Changed lines of the file:
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@@
 <parts>
 <part name="JP1" library="pinhead" deviceset="PINHD-1X8" device=""/>
-<part name="R1" library="resistor" deviceset="R-EU_" device="R0805" value="270E"/>
+<part name="R1" library="resistor" deviceset="R-EU_" device="R1206" value="270E"/>
 <part name="LED1" library="led" deviceset="LED" device="5MM"/>
 <part name="P+1" library="supply1" deviceset="+5V" device=""/>
 <part name="SUPPLY1" library="supply2" deviceset="GND" device=""/>
-<part name="R2" library="resistor" deviceset="R-EU_" device="R0805" value="270E"/>
-<part name="R3" library="resistor" deviceset="R-EU_" device="R0805" value="270E"/>
-<part name="R4" library="resistor" deviceset="R-EU_" device="R0805" value="270E"/>
-<part name="R5" library="resistor" deviceset="R-EU_" device="R0805" value="270E"/>
+<part name="R2" library="resistor" deviceset="R-EU_" device="R1206" value="270E"/>
+<part name="R3" library="resistor" deviceset="R-EU_" device="R1206" value="270E"/>
+<part name="R4" library="resistor" deviceset="R-EU_" device="R1206" value="270E"/>
+<part name="R5" library="resistor" deviceset="R-EU_" device="R1206" value="270E"/>
 <part name="LED2" library="led" deviceset="LED" device="5MM"/>
 <part name="LED3" library="led" deviceset="LED" device="5MM"/>
