File: Electronic Design/Eagle Files & BOMs/Main_board.brd (EAGLE design)
At the start: 99.9 x 69 mm, 43 parts, among them IC2 ATMEGA328-PU, IC3 LM2576S, Q1 IRF9540, Q2 IRF9540, X1 16MHz

Commit message: adding new layout of PCB
Parts:
- moved R10 271.8 mm to (43.6, 54.4)
- moved R9 264.3 mm to (43.7, 51.7), turned to 180 degrees
- moved C11 245.7 mm to (57.4, 44.4), turned to 90 degrees
- moved D3 239.5 mm to (52.0, 34.8), turned to 270 degrees
- moved C4 237.0 mm to (47.4, 53.0), turned to 90 degrees
- moved C5 220.8 mm to (52.2, 25.5), turned to 270 degrees
- moved C3 210.5 mm to (85.3, 32.9), turned to 180 degrees
- moved L1 183.9 mm to (83.2, 14.5), turned to 90 degrees
- moved D2 169.4 mm to (72.9, 11.7), turned to 270 degrees
- moved U$2 149.1 mm to (47.2, 42.4), turned to 180 degrees
- moved R8 124.3 mm to (48.4, 34.6), turned to 180 degrees
- moved R7 121.7 mm to (47.8, 37.7), turned to 180 degrees
- moved U$1 118.6 mm to (45.1, 24.8), turned to 180 degrees
- moved POT1 110.5 mm to (78.9, 24.8), turned to 90 degrees
- moved R3 98.9 mm to (73.1, 18.7), turned to 270 degrees
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Connections:
- new net BUTTON: IC2.4, R5.2, S2.4
- net N$8: no longer R5.2, S2.4
Routing:
- net M1S: track 0.00 -> 57.9 mm
- net N$8: track 33.4 -> 6.95 mm
- net N$19: track 53.9 -> 29.4 mm
- net N$14: track 19.8 -> 0.00 mm
- net N$10: track 65.0 -> 45.8 mm
- net IIN: track 0.06 -> 17.2 mm
- net N$26: track 0.00 -> 14.6 mm
- net BUTTON: track 0.00 -> 13.5 mm
- net +5V: track 117.3 -> 104.0 mm
- net N$7: track 14.4 -> 26.4 mm
- net N$23: track 0.00 -> 7.74 mm
- net VIN: track 16.4 -> 23.5 mm
- net N$4: track 10.4 -> 15.9 mm
- net N$18: track 33.7 -> 39.0 mm
- net N$35: track 24.0 -> 20.3 mm
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- added copper zone on layer 1, net N$13
- added copper zone on layer 1, net N$24
Other:
- board size 99.9 x 69 mm -> 100 x 63.5 mm
