File: Electronic Design/Eagle Files & BOMs/Main_board.brd (EAGLE design)
At the start: 90 x 60 mm, 52 parts, among them IC2 ATMEGA328-PU, IC3 LM2576S, Q1 BSS192P, Q2 FQD7P20, X1 16MHz

Commit message: Tidying up ground planes and traces. Adding ground stitching vias
Parts:
- moved R9 2.55 mm to (44.4, 34.7), turned to 0 degrees
- moved C12 0.40 mm to (25.6, 30.7), turned to 0 degrees
Routing:
- net VIN_CURRENT_MEASURED: track 43.4 -> 50.2 mm
- net VIN: track 38.9 -> 38.1 mm
- net GND: vias 27 -> 32
Changed lines of the file:
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@@
 <element name="C11" library="resistor" package="C1206K" value="10n" x="57.45" y="35.34" rot="R90"/>
 <element name="D3" library="diode" package="DO35Z10" value="5.1V" x="65.28" y="32.85" rot="MR270"/>
-<element name="R9" library="resistor" package="R0805" value="21k5" x="42.52" y="36.36" rot="R90"/>
+<element name="R9" library="resistor" package="R0805" value="21k5" x="44.44" y="34.68"/>
 <element name="R10" library="resistor" package="R0805" value="1k13" x="44.45" y="32.9" rot="MR180"/>
 <element name="D4" library="diode" package="DO35Z10" value="5.1V" x="80.93" y="21.5" rot="R270"/>
@@
 <attribute name="OC_FARNELL" value="unknown" x="6.85" y="40.8" size="1.778" layer="27" rot="R90" display="off"/>
 </element>
-<element name="C12" library="resistor" package="E3,5-8" value="100uF" x="25.22" y="30.64" rot="R180"/>
+<element name="C12" library="resistor" package="E3,5-8" value="100uF" x="25.61" y="30.74"/>
 <element name="C13" library="resistor" package="C1206K" value="0.1u" x="28.67" y="22.86" rot="R90"/>
 </elements>
@@
 <wire x1="45.4" y1="32.9" x2="53.70568125" y2="32.9" width="0.6096" layer="16"/>
 <wire x1="53.70568125" y1="32.9" x2="57.373834375" y2="36.568153125" width="0.6096" layer="16"/>
-<wire x1="42.52" y1="35.41" x2="42.52" y2="31.08" width="0.6096" layer="1"/>
-<wire x1="42.52" y1="31.08" x2="43.17" y2="30.43" width="0.6096" layer="1"/>
 <wire x1="43.17" y1="30.43" x2="43.2" y2="30.43" width="0.6096" layer="1"/>
-<wire x1="43.2" y1="30.43" x2="43.44" y2="30.19" width="0.6096" layer="1"/>
+<wire x1="43.44" y1="30.19" x2="43.2" y2="30.43" width="0.6096" layer="1"/>
 <via x="43.44" y="30.19" extent="1-16" drill="0.6" shape="square"/>
 <wire x1="43.44" y1="30.19" x2="44" y2="30.19" width="0.6096" layer="16"/>
@@
 <wire x1="57.373834375" y1="36.568153125" x2="60.7573125" y2="36.568153125" width="0.6096" layer="16"/>
 <wire x1="60.7573125" y1="36.568153125" x2="60.9225375" y2="36.402928125" width="0.6096" layer="16"/>
+<wire x1="43.49" y1="34.68" x2="43.49" y2="30.24" width="0.6096" layer="1"/>
+<wire x1="43.49" y1="30.24" x2="43.44" y2="30.19" width="0.6096" layer="1"/>
 </signal>
 <signal name="IIN">
@@
 <via x="17.52569375" y="48.3202" extent="1-16" drill="0.6" shape="square"/>
 <via x="39.98569375" y="11.7502" extent="1-16" drill="0.6" shape="square"/>
-<via x="20.0898" y="30.56569375" extent="1-16" drill="0.6" shape="square"/>
+<via x="27.2198" y="28.29569375" extent="1-16" drill="0.6" shape="square"/>
 <via x="75.35569375" y="38.8602" extent="1-16" drill="0.6" shape="square"/>
 <via x="79.71569375" y="43.5402" extent="1-16" drill="0.6" shape="square"/>
@@
 <via x="78.58569375" y="16.6602" extent="1-16" drill="0.6" shape="square"/>
 <via x="36.5902" y="13.86430625" extent="1-16" drill="0.6" shape="square"/>
-<via x="29.3102" y="30.93430625" extent="1-16" drill="0.6" shape="square"/>
+<via x="28.7202" y="33.08430625" extent="1-16" drill="0.6" shape="square"/>
 <contactref element="R5" pad="1"/>
 <contactref element="PROGAMMING_HEADER" pad="6"/>
-<via x="23.3098" y="32.90569375" extent="1-16" drill="0.6" shape="square"/>
+<via x="20.7698" y="38.68569375" extent="1-16" drill="0.6" shape="square"/>
 <polygon width="0.8128" layer="16" rank="2">
 <vertex x="0.03" y="58.94"/>
@@
 <contactref element="C10" pad="2"/>
 <contactref element="C6" pad="2"/>
-<via x="29.16569375" y="33.3802" extent="1-16" drill="0.6" shape="square"/>
+<via x="29.29569375" y="30.7202" extent="1-16" drill="0.6" shape="square"/>
 <via x="71.63569375" y="33.7702" extent="1-16" drill="0.6" shape="square"/>
 <contactref element="ATMEGA_DIO" pad="7"/>
@@
 <contactref element="AIO" pad="6"/>
 <via x="43.23569375" y="25.7302" extent="1-16" drill="0.6" shape="square"/>
-<via x="85.9698" y="17.70569375" extent="1-16" drill="0.6" shape="square"/>
+<via x="75.7098" y="18.46569375" extent="1-16" drill="0.6" shape="square"/>
 <contactref element="D4" pad="A"/>
 <contactref element="R12" pad="1"/>
-<via x="33.2498" y="35.76569375" extent="1-16" drill="0.6" shape="square"/>
+<via x="32.0498" y="36.18569375" extent="1-16" drill="0.6" shape="square"/>
 <via x="48.0698" y="56.81569375" extent="1-16" drill="0.6" shape="square"/>
 <via x="48.6998" y="50.34569375" extent="1-16" drill="0.6" shape="square"/>
 <via x="47.7898" y="52.38569375" extent="1-16" drill="0.6" shape="square"/>
 <via x="46.3598" y="47.56569375" extent="1-16" drill="0.6" shape="square"/>
-<via x="38.00569375" y="35.7402" extent="1-16" drill="0.6" shape="square"/>
+<via x="41.10569375" y="36.1102" extent="1-16" drill="0.6" shape="square"/>
 <contactref element="C12" pad="-"/>
 <contactref element="C13" pad="2"/>
@@
 <contactref element="LED2" pad="C"/>
 <contactref element="C3" pad="-"/>
-<via x="23.3498" y="28.20569375" extent="1-16" drill="0.6" shape="square"/>
+<via x="18.4498" y="35.16569375" extent="1-16" drill="0.6" shape="square"/>
 <via x="29.0802" y="26.56430625" extent="1-16" drill="0.6" shape="square"/>
 <wire x1="49.17" y1="43.75" x2="49.17" y2="44.75549375" width="0.6096" layer="1"/>
@@
 <wire x1="59.44" y1="38.83" x2="60.809609375" y2="38.83" width="0.6096" layer="1"/>
 <wire x1="60.809609375" y1="38.83" x2="60.9225375" y2="38.942928125" width="0.6096" layer="1"/>
+<polygon width="0.6096" layer="1">
+<vertex x="27.06" y="25.44"/>
+<vertex x="30.3" y="25.44"/>
+<vertex x="30.36" y="25.44"/>
+<vertex x="30.36" y="22.91"/>
+<vertex x="27" y="22.91"/>
+<vertex x="27" y="25.38"/>
+</polygon>
+<via x="17.3298" y="25.18569375" extent="1-16" drill="0.6" shape="square"/>
+<via x="3.0898" y="14.59569375" extent="1-16" drill="0.6" shape="square"/>
+<via x="12.3198" y="11.10569375" extent="1-16" drill="0.6" shape="square"/>
+<via x="40.87569375" y="17.4002" extent="1-16" drill="0.6" shape="square"/>
+<via x="39.98569375" y="14.8302" extent="1-16" drill="0.6" shape="square"/>
 </signal>
 <signal name="VIN_CURRENT_MEASURED">
@@
 <contactref element="C12" pad="+"/>
 <contactref element="C13" pad="1"/>
-<wire x1="45.09" y1="40.73" x2="45.09" y2="39.47" width="2.1844" layer="1"/>
-<wire x1="43.33" y1="37.71" x2="45.09" y2="39.47" width="2.1844" layer="1"/>
-<wire x1="43.33" y1="37.71" x2="30.17" y2="37.71" width="2.1844" layer="1"/>
-<wire x1="30.17" y1="37.71" x2="27" y2="34.54" width="2.1844" layer="1"/>
-<wire x1="27" y1="34.54" x2="27" y2="30.642" width="2.1844" layer="1"/>
-<wire x1="27" y1="30.642" x2="26.998" y2="30.64" width="2.1844" layer="1"/>
 <polygon width="0.6096" layer="1" thermals="no">
 <vertex x="44.07" y="41.8"/>
@@
 </polygon>
 <contactref element="R9" pad="2"/>
-<wire x1="42.52" y1="37.31" x2="42.93" y2="37.31" width="0.6096" layer="1"/>
-<wire x1="42.93" y1="37.31" x2="43.33" y2="37.71" width="0.6096" layer="1"/>
-<wire x1="26.998" y1="30.64" x2="26.998" y2="27.338" width="2.1844" layer="1"/>
-<wire x1="26.998" y1="27.338" x2="24.88" y2="25.22" width="2.1844" layer="1"/>
-<wire x1="24.88" y1="25.22" x2="24.88" y2="22.46" width="2.1844" layer="1"/>
-<wire x1="24.88" y1="22.46" x2="25.92" y2="21.42" width="2.1844" layer="1"/>
-<wire x1="25.92" y1="21.42" x2="28.61" y2="21.42" width="2.1844" layer="1"/>
-<wire x1="28.61" y1="21.42" x2="28.67" y2="21.36" width="2.1844" layer="1"/>
 <wire x1="28.67" y1="21.36" x2="31.84" y2="21.36" width="2.1844" layer="1"/>
 <wire x1="31.84" y1="21.36" x2="31.9" y2="21.42" width="2.1844" layer="1"/>
 <wire x1="31.84" y1="21.36" x2="32.4304" y2="21.36" width="0.6096" layer="1"/>
 <wire x1="32.4304" y1="21.36" x2="32.4328" y2="21.3576" width="0.6096" layer="1"/>
+<wire x1="45.09" y1="40.73" x2="45.1" y2="40.73" width="2.1844" layer="1"/>
+<wire x1="45.1" y1="40.73" x2="45.1" y2="38.32" width="2.1844" layer="1"/>
+<wire x1="42.52" y1="38.32" x2="45.1" y2="38.32" width="2.1844" layer="1"/>
+<wire x1="42.52" y1="38.32" x2="29.84" y2="38.32" width="2.1844" layer="1"/>
+<wire x1="29.84" y1="38.32" x2="23.85" y2="32.33" width="2.1844" layer="1"/>
+<wire x1="23.85" y1="32.33" x2="23.85" y2="30.758" width="2.1844" layer="1"/>
+<wire x1="23.85" y1="30.758" x2="23.832" y2="30.74" width="2.1844" layer="1"/>
+<wire x1="45.39" y1="34.68" x2="42.52" y2="38.32" width="0.6096" layer="1"/>
+<wire x1="23.832" y1="30.74" x2="23.832" y2="21.708" width="2.1844" layer="1"/>
+<wire x1="23.832" y1="21.708" x2="24.14" y2="21.4" width="2.1844" layer="1"/>
+<wire x1="24.14" y1="21.4" x2="28.63" y2="21.4" width="2.1844" layer="1"/>
+<wire x1="28.63" y1="21.4" x2="28.67" y2="21.36" width="2.1844" layer="1"/>
 </signal>
 <signal name="VIN_PROTECTED">
@@
 <wire x1="36.59" y1="7.822" x2="44.128" y2="7.822" width="2.1844" layer="1"/>
 <wire x1="44.128" y1="7.822" x2="46.69" y2="5.26" width="2.1844" layer="1"/>
-<wire x1="46.69" y1="5.26" x2="46.69" y2="3.51" width="2.1844" layer="1"/>
-<wire x1="46.69" y1="3.51" x2="47.71" y2="2.49" width="2.1844" layer="1"/>
-<wire x1="47.71" y1="2.49" x2="55.78221875" y2="2.49" width="2.1844" layer="1"/>
-<wire x1="55.78221875" y1="2.49" x2="60.522215625" y2="7.229996875" width="2.1844" layer="1"/>
+<wire x1="46.69" y1="5.26" x2="46.69" y2="3.51" width="2.1844" layer="16"/>
+<wire x1="46.69" y1="3.51" x2="47.71" y2="2.49" width="2.1844" layer="16"/>
+<wire x1="47.71" y1="2.49" x2="55.78221875" y2="2.49" width="2.1844" layer="16"/>
+<wire x1="55.78221875" y1="2.49" x2="60.522215625" y2="7.229996875" width="2.1844" layer="16"/>
 </signal>
 <signal name="N$18">
