File: Electronic Design/Eagle Files & BOMs/Main_board.sch (EAGLE design)
At the start: 49 parts, among them IC2 ATMEGA328-PU, IC3 LM2576S, Q1 IRF9540, Q2 IRF9540, X1 16MHz

Commit message: Adding new overvoltage protection FETs and renaming nets
Parts:
- Q1: value IRF9540 -> BSS192P; device transistor-power:PMOSFET_PTO220BH -> Samson:BSS192P
- Q2: value IRF9540 -> FQD7P20; device transistor-power:PMOSFET_PTO220BH -> Samson:FQD7P20
- R1: value 1k -> 100k; device resistor:R-EU_VTA52 -> resistor:R-EU_0207/10
Connections:
- net M1S renamed VIN_CURRENT_MEASURED
- net N$1 renamed VIN_AC1
- net N$10 renamed VIN_UNPROTECTED
- net N$11 renamed D11
- net N$12 renamed D12
- net N$13 renamed BUCK_OUTPUT
- net N$15 renamed CRYSTAL2
- net N$16 renamed CRYSTAL1
- net N$17 renamed RESET
- net N$19 renamed VIN_AC2
- net N$2 renamed VOUT_PREFUSE
- net N$20 renamed D8
- net N$21 renamed D7
- net N$22 renamed D6
- net N$24 renamed VOUT_FINAL
- net N$25 renamed D5
- net N$26 renamed BUCK_FEEDBACK
- net N$3 renamed VIN_PROTECTED
- net N$35 renamed Q2_GATE
- net N$6 renamed D9
- net N$7 renamed Q1_GATE
- net N$8 renamed D13
- net N$9 renamed D10
Changed lines of the file:
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@@
 <part name="C1" library="resistor" deviceset="C-EU" device="C1206K" value="10n"/>
 <part name="C2" library="resistor" deviceset="CPOL-EU" device="E3.5-10" value="220uF"/>
-<part name="Q1" library="transistor-power" deviceset="PMOSFET_P" device="TO220BH" value="IRF9540"/>
-<part name="Q2" library="transistor-power" deviceset="PMOSFET_P" device="TO220BH" value="IRF9540"/>
 <part name="POT3" library="resistor" deviceset="R-TRIMM" device="3296W" value="5k"/>
-<part name="R1" library="resistor" deviceset="R-EU_" device="VTA52" value="1k"/>
+<part name="R1" library="resistor" deviceset="R-EU_" device="0207/10" value="100k"/>
 <part name="SUPPLY22" library="supply2" deviceset="GND" device=""/>
 <part name="SUPPLY23" library="supply2" deviceset="GND" device=""/>
@@
 <part name="R12" library="resistor" deviceset="R-EU_" device="R1206" value="2k"/>
 <part name="SUPPLY15" library="supply2" deviceset="GND" device=""/>
+<part name="Q1" library="Samson" deviceset="BSS192P" device=""/>
+<part name="Q2" library="Samson" deviceset="FQD7P20" device=""/>
 </parts>
 <sheets>
@@
 <instance part="C1" gate="G$1" x="-1.27" y="74.93"/>
 <instance part="C2" gate="G$1" x="-31.75" y="78.74"/>
-<instance part="Q1" gate="G$1" x="-54.61" y="81.28"/>
-<instance part="Q2" gate="G$1" x="-41.91" y="86.36" rot="R90"/>
 <instance part="POT3" gate="G$1" x="-66.04" y="83.82"/>
 <instance part="R1" gate="G$1" x="-49.53" y="71.12" rot="R90"/>
@@
 <instance part="R12" gate="G$1" x="138.43" y="33.02" rot="R90"/>
 <instance part="SUPPLY15" gate="GND" x="138.43" y="24.13"/>
+<instance part="Q1" gate="G$1" x="-52.07" y="81.28" rot="MR180"/>
+<instance part="Q2" gate="G$1" x="-41.91" y="86.36" rot="R90"/>
 </instances>
 <busses>
@@
 </segment>
 </net>
-<net name="M1S" class="0">
+<net name="VIN_CURRENT_MEASURED" class="0">
 <segment>
 <wire x1="60.96" y1="88.9" x2="60.96" y2="48.26" width="0.1524" layer="91"/>
@@
 </segment>
 </net>
-<net name="N$3" class="0">
-<segment>
-<pinref part="Q2" gate="G$1" pin="D"/>
+<net name="VIN_PROTECTED" class="0">
+<segment>
 <wire x1="-36.83" y1="88.9" x2="-31.75" y2="88.9" width="0.1524" layer="91"/>
 <pinref part="C2" gate="G$1" pin="+"/>
@@
 <pinref part="R9" gate="G$1" pin="2"/>
 <junction x="-16.51" y="88.9"/>
-</segment>
-</net>
-<net name="N$10" class="0">
-<segment>
-<pinref part="Q1" gate="G$1" pin="S"/>
+<pinref part="Q2" gate="G$1" pin="D"/>
+</segment>
+</net>
+<net name="VIN_UNPROTECTED" class="0">
+<segment>
 <wire x1="-52.07" y1="86.36" x2="-52.07" y2="88.9" width="0.1524" layer="91"/>
-<pinref part="Q2" gate="G$1" pin="S"/>
 <wire x1="-52.07" y1="88.9" x2="-46.99" y2="88.9" width="0.1524" layer="91"/>
 <pinref part="POT3" gate="G$1" pin="E"/>
@@
 <wire x1="-78.74" y1="88.9" x2="-66.04" y2="88.9" width="0.1524" layer="91"/>
 <junction x="-66.04" y="88.9"/>
-</segment>
-</net>
-<net name="N$35" class="0">
-<segment>
-<pinref part="Q1" gate="G$1" pin="D"/>
+<pinref part="Q1" gate="G$1" pin="S"/>
+<pinref part="Q2" gate="G$1" pin="S"/>
+</segment>
+</net>
+<net name="Q2_GATE" class="0">
+<segment>
 <pinref part="R1" gate="G$1" pin="2"/>
 <wire x1="-52.07" y1="76.2" x2="-49.53" y2="76.2" width="0.1524" layer="91"/>
 <wire x1="-49.53" y1="76.2" x2="-44.45" y2="76.2" width="0.1524" layer="91"/>
-<pinref part="Q2" gate="G$1" pin="G"/>
 <wire x1="-44.45" y1="76.2" x2="-44.45" y2="81.28" width="0.1524" layer="91"/>
 <junction x="-49.53" y="76.2"/>
+<pinref part="Q1" gate="G$1" pin="D"/>
+<pinref part="Q2" gate="G$1" pin="G"/>
 </segment>
 </net>
@@
 </segment>
 </net>
-<net name="N$15" class="0">
+<net name="CRYSTAL2" class="0">
 <segment>
 <pinref part="X1" gate="G$1" pin="1"/>
@@
 </segment>
 </net>
-<net name="N$16" class="0">
+<net name="CRYSTAL1" class="0">
 <segment>
 <pinref part="X1" gate="G$1" pin="2"/>
@@
 </segment>
 </net>
-<net name="N$17" class="0">
+<net name="RESET" class="0">
 <segment>
 <pinref part="R4" gate="G$1" pin="2"/>
@@
 </segment>
 </net>
-<net name="N$8" class="0">
+<net name="D13" class="0">
 <segment>
 <pinref part="IC2" gate="1" pin="DIGITAL_13"/>
@@
 </segment>
 </net>
-<net name="N$6" class="0">
+<net name="D9" class="0">
 <segment>
 <pinref part="IC2" gate="1" pin="DIGITAL_9(PWM)"/>
@@
 </segment>
 </net>
-<net name="N$9" class="0">
+<net name="D10" class="0">
 <segment>
 <pinref part="ATMEGA_DIO" gate="A" pin="2"/>
@@
 </segment>
 </net>
-<net name="N$11" class="0">
+<net name="D11" class="0">
 <segment>
 <pinref part="IC2" gate="1" pin="DIGITAL_11(PWM)"/>
@@
 </segment>
 </net>
-<net name="N$12" class="0">
+<net name="D12" class="0">
 <segment>
 <pinref part="IC2" gate="1" pin="DIGITAL_12"/>
@@
 </segment>
 </net>
-<net name="N$7" class="0">
-<segment>
+<net name="Q1_GATE" class="0">
+<segment>
+<pinref part="POT3" gate="G$1" pin="S"/>
+<wire x1="-57.15" y1="83.82" x2="-60.96" y2="83.82" width="0.1524" layer="91"/>
 <pinref part="Q1" gate="G$1" pin="G"/>
-<pinref part="POT3" gate="G$1" pin="S"/>
-<wire x1="-60.96" y1="83.82" x2="-59.69" y2="83.82" width="0.1524" layer="91"/>
-</segment>
-</net>
-<net name="N$19" class="0">
+</segment>
+</net>
+<net name="VIN_AC2" class="0">
 <segment>
 <pinref part="VIN" gate="A" pin="1"/>
@@
 </segment>
 </net>
-<net name="N$20" class="0">
+<net name="D8" class="0">
 <segment>
 <pinref part="IC2" gate="1" pin="DIGITAL_8"/>
@@
 </segment>
 </net>
-<net name="N$21" class="0">
+<net name="D7" class="0">
 <segment>
 <pinref part="IC2" gate="1" pin="DIGITAL_7"/>
@@
 </segment>
 </net>
-<net name="N$22" class="0">
+<net name="D6" class="0">
 <segment>
 <pinref part="IC2" gate="1" pin="DIGITAL_6(PWM)"/>
@@
 </segment>
 </net>
-<net name="N$25" class="0">
+<net name="D5" class="0">
 <segment>
 <pinref part="IC2" gate="1" pin="DIGITAL_5(PWM)"/>
@@
 </segment>
 </net>
-<net name="N$13" class="0">
+<net name="BUCK_OUTPUT" class="0">
 <segment>
 <pinref part="L1" gate="G$1" pin="1"/>
@@
 </segment>
 </net>
-<net name="N$24" class="0">
+<net name="VOUT_FINAL" class="0">
 <segment>
 <pinref part="C3" gate="G$1" pin="+"/>
@@
 </segment>
 </net>
-<net name="N$26" class="0">
+<net name="BUCK_FEEDBACK" class="0">
 <segment>
 <pinref part="POT1" gate="G$1" pin="S"/>
@@
 </segment>
 </net>
-<net name="N$1" class="0">
+<net name="VIN_AC1" class="0">
 <segment>
 <pinref part="VIN" gate="A" pin="3"/>
@@
 </segment>
 </net>
-<net name="N$2" class="0">
+<net name="VOUT_PREFUSE" class="0">
 <segment>
 <pinref part="POT1" gate="G$1" pin="A"/>
