File: Electronic Design - TH/Eagle Files & BOMs/Main_board.brd (EAGLE design)
At the start: 90 x 60 mm, 46 parts, among them IC2 ATMEGA328-PU, Q1 BSS192P, Q2 FQD7P20, X1 16MHz

Commit message: replaced SMD resistors, caps and MOSFETs with TH components
Parts:
- C1, C10, C11, C4, C5, C6, C7: device resistor:C1206K -> resistor:C050-024X044
- C8, C9: device resistor:C0805K -> resistor:C050-024X044
- PWR, UC_PWR: device adafruit:1206 -> led:LED3MM
- Q1: value BSS192P -> (none); device Samson:BSS192P -> Samson:TO220BH
- Q2: value FQD7P20 -> (none); device Samson:TO252 -> Samson:TO220BH
- R10, R9: device resistor:R0805 -> resistor:0207/10
- R11, R12, R4, R5, R7, R8: device resistor:R1206 -> resistor:0207/10
- R2: device resistor:M1206 -> resistor:0207/15
- U$1: device Samson:TO220BH -> Samson:TO220BH2
Connections:
- net GND: now also PWR.K; no longer PWR.C
- net N$28: now also UC_PWR.K; no longer UC_PWR.C
- net Q1_GATE: now also Q1.G; no longer Q1.1
- net Q2_GATE: now also Q1.S, Q2.G; no longer Q1.2, Q1.4, Q2.1, R1.2
- net VIN_PROTECTED: now also Q2.D; no longer Q2.3
- net VIN_UNPROTECTED: now also Q1.D, Q2.S; no longer Q1.3, Q2.2
Routing:
- net VIN_CURRENT_MEASURED: track 62.8 -> 0.00 mm, vias 1 -> 0
- net VIN_AC2: track 46.2 -> 0.00 mm
- net +5V: track 118.3 -> 90.0 mm, vias 1 -> 0
- net VIN_AC1: track 23.8 -> 0.00 mm
- net VIN_PROTECTED: track 22.0 -> 0.00 mm
- net VIN_UNPROTECTED: track 23.2 -> 3.69 mm
- net IIN: track 23.7 -> 10.6 mm
- net Q1_GATE: track 12.0 -> 0.00 mm
- net Q2_GATE: track 9.18 -> 0.00 mm
- net N$28: track 4.40 -> 11.6 mm
- net N$1: track 6.63 -> 0.00 mm
- net N$23: track 6.60 -> 12.2 mm
- net GND: track 9.32 -> 3.73 mm, vias 25 -> 24
- net VIN: track 31.4 -> 35.8 mm
- net CRYSTAL1: track 8.62 -> 11.6 mm
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
Commit message: correcting mosfet postion
Connections:
- net Q2_GATE: now also Q1.D, R1.2; no longer Q1.S
- net VIN_UNPROTECTED: now also Q1.S; no longer Q1.D
Changed lines of the file:
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@@
 <contactref element="Q2" pad="S"/>
 <wire x1="31.495396875" y1="56.51505" x2="35.18505" y2="56.51505" width="0.8128" layer="1"/>
-<contactref element="Q1" pad="D"/>
-<wire x1="35.18505" y1="56.51505" x2="36.85" y2="61.28" width="0" layer="19" extent="1-1"/>
+<contactref element="Q1" pad="S"/>
+<wire x1="35.18505" y1="56.51505" x2="34.31" y2="61.28" width="0" layer="19" extent="1-1"/>
 <wire x1="31.61" y1="52.38" x2="31.495396875" y2="56.51505" width="0" layer="19" extent="1-1"/>
 <wire x1="26.750996875" y1="39.824584375" x2="31.61" y2="52.38" width="0" layer="19" extent="1-1"/>
 </signal>
 <signal name="Q2_GATE">
-<contactref element="Q2" pad="G"/>
 <polygon width="0.8128" layer="1" thermals="no">
 <vertex x="39.77" y="54.96"/>
@@
 <vertex x="34.51" y="54.96"/>
 </polygon>
-<contactref element="Q1" pad="S"/>
-<wire x1="36.69" y1="52.38" x2="34.31" y2="61.28" width="0" layer="19" extent="1-1"/>
+<contactref element="Q1" pad="D"/>
+<contactref element="Q2" pad="G"/>
+<contactref element="R1" pad="2"/>
+<wire x1="40.79703125" y1="57.813271875" x2="36.85" y2="61.28" width="0" layer="19" extent="1-1"/>
+<wire x1="36.69" y1="52.38" x2="40.79703125" y2="57.813271875" width="0" layer="19" extent="1-1"/>
 </signal>
 <signal name="+5V">
