File: Electronic Design - TH/Eagle Files & BOMs/Main_board_TH.brd (EAGLE design)
At the start: 90 x 60 mm, 41 parts, among them M1 ARDUINO-NANO-3.0, Q1 IRF9520, Q2 IRF9520

Commit message: Removed: pin headers for arduino, button for arduino and LED for LM2596. Inital board layout complete. Sub modules pretty much done but overall layout still needs work
Parts:
- removed C5: 0.1u, resistor:C050-024X044
- removed JP1: (no value), pinhead:1X06
- removed PWR: (no value), led:LED3MM
- removed R11: 2k, resistor:0207/10
- removed R5: 10k, resistor:0207/10
- removed S2: (no value), switch-omron:B3F-10XX
- removed U$1: LM317, Samson:TO220BH2
- removed U$2: LM358, Samson:DIL08
- added C4: 10u, resistor:E2,5-7
- added D2: 5.1V, diode:DO35Z10
- added LM317: LM317, Samson:TO220BV
- added LM358: LM358, Samson:DIL08
- B1: value KBPC610 -> GBU406; device rectifier:GBPC6 -> rectifier:GBU4S
- C10, C3: device resistor:C050-024X044 -> resistor:E2,5-7
- Q1, Q2: device Samson:TO220BH -> Samson:TO220BV
- moved C3 212.8 mm to (57.2, 37.1), turned to 90 degrees
- moved R16 187.6 mm to (37.5, 44.5), turned to 180 degrees
- moved R15 165.2 mm to (29.8, 36.4), turned to 270 degrees
- moved R14 152.6 mm to (32.6, 36.3), turned to 90 degrees
- moved R13 152.2 mm to (51.6, 44.4), turned to 180 degrees
- moved VIN 126.5 mm to (43.2, 141.9), turned to 0 degrees
- moved R4 118.0 mm to (37.5, 47.0), turned to 180 degrees
- moved R3 110.6 mm to (51.6, 47.2), turned to 180 degrees
- moved B1 87.2 mm to (43.4, 129.7), turned to 180 degrees
- moved Q2 85.3 mm to (74.5, 121.1), turned to 0 degrees
- moved D4 84.8 mm to (13.5, 73.0), turned to 180 degrees
- moved R12 75.3 mm to (13.5, 70.0), turned to 0 degrees
- moved F2 74.5 mm to (15.3, 114.8), turned to 270 degrees
- moved Q1 71.0 mm to (62.5, 121.1), turned to 0 degrees
- moved R1 69.8 mm to (68.2, 124.0)
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Connections:
- net N$2 renamed A4
- net N$3 renamed A5
- removed net 5V: M1.J2.4
- removed net BUTTON: M1.J1.5, R5.2, S2.4
- removed net N$18: PWR.A, R11.1
- removed net N$28: R12.2, UC_PWR.K
- removed net VIN_AC1: B1.AC1, F2.2, R6.1
- removed net VIN_AC2: B1.AC2, R6.2, VIN.1
- new net N$10: D5.A, U$3.OUT-, VOUT.3
- new net N$2: R12.1, UC_PWR.A
- new net N$7: B1.AC1, VIN.1
- new net N$9: B1.AC2, VIN.3
- net +5V: now also C10.+, LM317.2, M1.J2.4, R12.2; no longer C10.1, C5.1, M1.J2.1, S2.2, U$1.2, UC_PWR.A
- net A2: no longer JP1.1
- net A3: no longer JP1.2
- net A6: no longer JP1.3
- net A7: no longer JP1.4
- net GND: now also C10.-, C3.-, C4.-, D2.A, LM358.4, R6.2, UC_PWR.K; no longer C10.2, C3.2, C5.2, D5.A, JP1.5, JP1.6, PWR.K, R12.1, R5.1, U$2.4, U$3.OUT-, VOUT.3
- net IIN: now also D2.C, LM358.1; no longer U$2.1
- net N$1: now also B1.+; no longer VIN.3
- net N$23: now also LM317.1; no longer U$1.1
- net N$5: now also LM358.3; no longer U$2.3
- net N$6: now also LM358.2; no longer U$2.2
- net Q1_GATE: now also Q1.1; no longer Q1.G
- net Q2_GATE: now also Q1.2, Q2.1; no longer Q1.D, Q2.G
- net VIN: now also M1.J2.1
- net VIN_PROTECTED: now also C3.+, C4.+, LM317.3, LM358.8, Q2.2; no longer C3.1, Q2.D, U$1.3, U$2.8
- net VIN_UNPROTECTED: now also F2.2, Q1.3, Q2.3, R6.1; no longer B1.+, Q1.S, Q2.S
- net VOUT_FINAL: no longer R11.2
Routing:
- net VIN_PROTECTED: track 0.00 -> 84.6 mm
- net +5V: track 80.9 -> 1.95 mm
- net VIN_UNPROTECTED: track 3.69 -> 78.5 mm
- net GND: track 0.00 -> 61.9 mm, vias 24 -> 10
- net VOUT_FINAL: track 37.3 -> 0.00 mm
- net IIN: track 0.00 -> 37.0 mm
- net VIN: track 34.3 -> 0.00 mm
- net Q2_GATE: track 0.00 -> 22.2 mm
- net VOUT_PREFUSE: track 21.0 -> 0.00 mm
- net N$6: track 0.00 -> 15.6 mm
- net Q1_GATE: track 0.00 -> 15.2 mm
- net N$7: track 0.00 -> 12.3 mm
- net N$9: track 0.00 -> 12.3 mm
- net N$23: track 12.2 -> 0.00 mm
- net N$28: track 11.6 -> 0.00 mm
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- removed copper zone on layer 1, net BUCK_OUTPUT
- removed copper zone on layer 1, net GND
- removed copper zone on layer 16, net GND
- removed copper zone on layer 1, net Q2_GATE
- removed copper zone on layer 1, net VIN_PROTECTED
Other:
- board size 90 x 60 mm -> 86.2 x 145.6 mm
- board text added: "=>"
- board text added: "Active protection"
- board text added: "Connect your load here =>"
- board text added: "Connect your voltage supply here =>"
- board text added: "Current Measurement"
- board text added: "Input voltage smoothing"
- board text added: "Main power supply"
- board text added: "Passive protection"
- board text added: "Rectification"
- board text added: "Voltage Measurement"
- board text added: "uC Power Supply"
- board text removed: "_"

Commit message: high level layout complete and adding in BOM
Parts:
- moved SCREEN_OUT 46.2 mm to (45.7, 35.3)
- moved D5 46.1 mm to (79.6, 47.5)
- moved U$3 43.6 mm to (78.5, 72.7)
- moved F1 40.1 mm to (79.6, 29.3), turned to 270 degrees
- moved C1 39.3 mm to (41.0, 87.2), turned to 90 degrees
- moved D1 25.3 mm to (52.7, 82.8)
- moved R9 24.6 mm to (53.0, 90.5)
- moved R10 24.6 mm to (52.6, 86.8)
- moved C3 19.7 mm to (59.8, 56.6)
- moved D2 19.7 mm to (38.4, 56.1)
- moved LM358 19.7 mm to (47.1, 56.1)
- moved R13 19.7 mm to (54.2, 64.0)
- moved R14 19.7 mm to (35.1, 55.9)
- moved R15 19.7 mm to (32.3, 55.9)
- moved R2 19.7 mm to (47.0, 69.9)
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Connections:
- removed net A6: M1.J2.6
- removed net A7: M1.J2.5
- removed net IIN: D2.C, LM358.1, M1.J2.12, R13.1
- new net A0: D2.C, M1.J2.12
- new net A1: M1.J2.11
- new net I_IN: LM358.1, M1.J2.6, R13.1
- new net V_IN: C1.1, D1.C, M1.J2.5, R10.2, R9.1
- net VIN: no longer C1.1, D1.C, M1.J2.11, R10.2, R9.1
Routing:
- net VIN_PROTECTED: track 84.6 -> 14.4 mm
- net VIN_UNPROTECTED: track 78.5 -> 25.8 mm
- net IIN: track 37.0 -> 0.00 mm
- net I_IN: track 0.00 -> 36.6 mm
- net N$9: track 12.3 -> 9.83 mm
- net N$7: track 12.3 -> 9.90 mm
Other:
- board size 86.2 x 145.6 mm -> 91.7 x 133.3 mm
- board text added: "Connect your voltage supply here"
- board text removed: "Connect your voltage supply here =>"
- board text removed: "Input voltage smoothing"

Commit message: completing passive protection and active protection alignment and renaming components sequentially (i.e. R1, R2, R3, ...)
Parts:
- removed C10: 10u, resistor:E2,5-7
- removed D5: 5.1V, diode:DO35Z10
- removed POT3: 100k, resistor:RTRIM3296W
- removed U$3: DC-DC-STEP-DOWN-LM2596, diy-modules:DC-DC-STEP-DOWN-LM2596
- added C5: 10n, resistor:C050-024X044
- added C6: 10u, resistor:E2,5-7
- added D3: 5.1V, diode:DO35Z10
- added LM2596_BUCK_CONVERTER: DC-DC-STEP-DOWN-LM2596, diy-modules:DC-DC-STEP-DOWN-LM2596
- added R11: 1k, resistor:0207/10
- added R5: 10k, resistor:0207/10
- C1: value 10n -> 220uF; device resistor:C050-024X044 -> resistor:E3,5-10
- C2: value 220uF -> 10n; device resistor:E3,5-10 -> resistor:C050-024X044
- R1: value 100k -> S14K75; device resistor:0207/10 -> varistor:S14K17
- R10: value 1k -> 0R01; device resistor:0207/10 -> resistor:0207/15
- R12: value 2k -> 1k
- R14: value 10k -> 47k
- R16: value 47k -> 10k
- R2: value 0R01 -> 10k; device resistor:0207/15 -> resistor:0207/10
- R3: value 1k -> 10k
- R4: value 1k -> 100k
- R6: value S14K75 -> 1k; device varistor:S14K17 -> resistor:0207/10
- R9: value 10k -> 2k
- moved F2 105.0 mm to (79.6, 29.3)
- moved F1 102.8 mm to (13.4, 108.0)
- moved C2 72.7 mm to (26.8, 37.4), turned to 90 degrees
- moved D4 67.6 mm to (79.6, 47.5)
- moved R4 57.2 mm to (72.0, 114.1)
- moved C4 54.7 mm to (59.4, 55.2), turned to 90 degrees
- moved R2 54.5 mm to (69.4, 119.6), turned to 0 degrees
- moved R3 52.6 mm to (69.4, 117.1)
- moved C3 51.0 mm to (15.0, 81.0), turned to 180 degrees
- moved R9 50.0 mm to (14.3, 58.8)
- moved R1 49.4 mm to (25.4, 105.5), turned to 0 degrees
- moved R12 37.9 mm to (53.7, 65.3), turned to 180 degrees
- moved R6 35.3 mm to (44.7, 82.6), turned to 180 degrees
- moved C1 34.2 mm to (72.9, 99.4), turned to 180 degrees
- moved D2 24.7 mm to (14.3, 61.8), turned to 180 degrees
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Connections:
- removed net Q1_GATE: POT3.2, Q1.1
- new net N$3: Q1.1, R2.1, R3.2
- net +5V: now also C6.+, D2.C, R9.2; no longer C10.+, D4.C, R12.2
- net A0: no longer D2.C
- net GND: now also C1.-, C2.2, C5.2, C6.-, D3.A, R1.2, R12.2, R16.1, R3.1, R4.1, R6.1; no longer C1.2, C10.-, C2.-, D4.A, POT3.1, R1.1, R14.1, R2.1, R3.2, R6.2
- net I_IN: now also C5.1, D3.C
- net N$1: now also F1.1; no longer F2.1
- net N$10: now also D4.A, LM2596_BUCK_CONVERTER.OUT-; no longer D5.A, U$3.OUT-
- net N$2: now also R9.1; no longer R12.1
- net N$4: now also LM2596_BUCK_CONVERTER.IN-, R10.2, R11.2; no longer R2.2, R4.2, U$3.IN-
- net N$5: now also R11.1, R14.1; no longer R16.1, R4.1
- net N$6: now also R12.1; no longer R3.1
- net Q2_GATE: now also R4.2; no longer R1.2
- net VIN_PROTECTED: now also C1.+, LM2596_BUCK_CONVERTER.IN+, R5.2; no longer C2.+, R9.2, U$3.IN+
- net VIN_UNPROTECTED: now also F1.2, R1.1, R2.2; no longer F2.2, POT3.3, R6.1
- net VOUT_FINAL: now also D4.C, F2.2; no longer D5.C, F1.2
- net VOUT_PREFUSE: now also F2.1, LM2596_BUCK_CONVERTER.OUT+; no longer F1.1, U$3.OUT+
- net V_IN: now also C2.1, R5.1, R6.2; no longer C1.1, R10.2, R9.1
Routing:
- net GND: track 61.9 -> 0.00 mm, vias 10 -> 12
- net Q1_GATE: track 15.2 -> 0.00 mm
- net N$3: track 0.00 -> 12.1 mm
- net VIN_UNPROTECTED: track 25.8 -> 32.0 mm
- net Q2_GATE: track 22.2 -> 21.1 mm
Other:
- board size 91.7 x 133.3 mm -> 90 x 130 mm
